File: hardware/tardis-r2.sch (EAGLE design)
At the start: 91 parts, among them IC1 LM4864, IC2 LSM6DSOXTR, IC3 LM5166YDRCR, J1 MOLEX-53261-0871, Q1 2N7002, Q2 2N7002, Q3 2N7002, Q4 2N7002, Q5 2N7002

Commit message: - added revision description for eagle pcb - added full sound playback for tardis
Other:
- note added: "Revision 2 changes: - NRST is now reouted to ST-Link connector instead of NJTRST"
Changed lines of the file:
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@@
 <part name="GND36" library="voltage-ground" library_urn="urn:adsk.eagle:library:704746" deviceset="GND" device=""/>
 <part name="U$29" library="voltage-ground" library_urn="urn:adsk.eagle:library:704746" deviceset="NC" device=""/>
+<part name="FRAME3" library="frames" library_urn="urn:adsk.eagle:library:229" deviceset="A4L-LOC" device=""/>
 </parts>
 <sheets>
@@
 </nets>
 </sheet>
+<sheet>
+<plain>
+<text x="7.62" y="170.18" size="1.778" layer="97" align="top-left">Revision 2 changes:
+- NRST is now reouted to ST-Link connector instead of NJTRST</text>
+</plain>
+<instances>
+<instance part="FRAME3" gate="G$1" x="0" y="0" smashed="yes">
+<attribute name="DRAWING_NAME" x="217.17" y="15.24" size="2.54" layer="94"/>
+<attribute name="LAST_DATE_TIME" x="217.17" y="10.16" size="2.286" layer="94"/>
+<attribute name="SHEET" x="230.505" y="5.08" size="2.54" layer="94"/>
+</instance>
+</instances>
+<busses>
+</busses>
+<nets>
+</nets>
+</sheet>
